Commit message: feature: increase robot's base position (URDF file), reconfigure ur10e_rg2_moveit package, add table(using mesh) into planning scene as collision object in rviz, rewrite test_TrajectoryPlanner.launch

File: ROS/src/ur10e_rg2_moveit/config/gazebo_ur10e_robot_rg2.urdf (robot description, URDF)
Before this commit: robot ur10e_robot_rg2, 17 links, 16 joints
Joints:
- joint base_link-base_link_inertia: origin xyz=0 0 0 rpy=0 0 3.141592653589793 -> xyz=0 0 1 rpy=0 0 3.141592653589793

File: ROS/src/ur10e_rg2_urdf/urdf/ur10e_with_rg2.urdf (robot description, URDF)
Before this commit: robot ur10e_robot_rg2, 17 links, 16 joints
Joints:
- joint base_link-base_link_inertia: origin xyz=0 0 0 rpy=0 0 3.141592653589793 -> xyz=0 0 1 rpy=0 0 3.141592653589793

Commit message: update

File: ROS/src/ur10e_rg2_moveit/config/gazebo_ur10e_robot_rg2.urdf (robot description, URDF)
Before this commit: robot ur10e_robot_rg2, 17 links, 16 joints
Joints:
- joint base_link-base_fixed_joint: origin xyz=0 0 0 rpy=0 0 3.141592653589793 -> xyz=0 0 0 rpy=0 0 3.14159265359
- joint base_link-base_link_inertia: origin xyz=0 0 1 rpy=0 0 3.141592653589793 -> xyz=0 0 0 rpy=0 0 3.14159265359
- joint elbow_joint: limit lower=-3.141592653589793 upper=3.141592653589793 effort=150.0 velocity=3.141592653589793 -> lower=-3.14159265359 upper=3.14159265359 effort=150.0 velocity=3.14159265359
- joint shoulder_lift_joint: limit lower=-6.283185307179586 upper=6.283185307179586 effort=330.0 velocity=2.0943951023931953 -> lower=-6.28318530718 upper=6.28318530718 effort=330.0 velocity=2.09439510239
- joint shoulder_pan_joint: limit lower=-6.283185307179586 upper=6.283185307179586 effort=330.0 velocity=2.0943951023931953 -> lower=-6.28318530718 upper=6.28318530718 effort=330.0 velocity=2.09439510239
- joint wrist_1_joint: limit lower=-6.283185307179586 upper=6.283185307179586 effort=56.0 velocity=3.141592653589793 -> lower=-6.28318530718 upper=6.28318530718 effort=56.0 velocity=3.14159265359
- joint wrist_2_joint: limit lower=-6.283185307179586 upper=6.283185307179586 effort=56.0 velocity=3.141592653589793 -> lower=-6.28318530718 upper=6.28318530718 effort=56.0 velocity=3.14159265359; origin xyz=0 -0.11985 -2.458164590756244e-11 rpy=1.570796327 0 0 -> xyz=0 -0.11985 -2.45816459076e-11 rpy=1.570796327 0 0
- joint wrist_3_joint: limit lower=-6.283185307179586 upper=6.283185307179586 effort=56.0 velocity=3.141592653589793 -> lower=-6.28318530718 upper=6.28318530718 effort=56.0 velocity=3.14159265359; origin xyz=0 0.11655 -2.390480459346185e-11 rpy=1.570796326589793 3.141592653589793 3.141592653589793 -> xyz=0 0.11655 -2.39048045935e-11 rpy=1.57079632659 3.14159265359 3.14159265359

File: UnityProject/Assets/URDF/ur10e_with_rg2.urdf (robot description, URDF)
Before this commit: robot ur10e_robot_rg2, 17 links, 16 joints
Joints:
- joint base_link-base_link_inertia: origin xyz=0 0 1 rpy=0 0 3.141592653589793 -> xyz=0 0 0 rpy=0 0 3.141592653589793
